File: Electrical/MainBoard/MainBoard.sch (EAGLE design)
At the start: 121 parts, among them IC1 MEGA1284-P, IC2 MCP4922-E/SL, IC3 MCP4921-E/SN, IC4 TL074D, IC5 TL074D, IC6 FT232RL, Q1 BC140-10, Q2 BC160, Q3 BC140-10, Q4 BC160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

Commit message: Modified DMM circuit to use DMMRectifier PCB
Parts:
- removed D8, D9: 5V, diode:ZENER-DIODESOD80C
- removed R35, R37: 100k, OwnDevices:R-EU_R0805
- removed R36, R38: 24k, OwnDevices:R-EU_R0805
- added DMM1_NEG, DMM2_NEG: (no value), OwnDevices:2,54/1,0
Connections:
- removed net DVM1_ADC: D8.C, IC1.(ADC6)PA6, R35.1, R36.2
- removed net DVM2_ADC: D9.C, IC1.(ADC7)PA7, R37.1, R38.2
- removed net N$40: DMM1.P, R35.2
- removed net N$41: DMM2.P, R37.2
- new net DMM1: DMM1.P, IC1.(ADC6)PA6
- new net DMM1_NEG: DMM1_NEG.P, IC1.(OC1A)PD5
- new net DMM2: DMM2.P, IC1.(ADC7)PA7
- new net DMM2_NEG: DMM2_NEG.P, IC1.(ICP)PD6
- net GND: no longer D8.A, D9.A, R36.1, R38.1
Other:
- note added: "DMM1 & DMM2 input range: 0 .. 5 V DMM1_NEG & DMM2_NEG indicate a negative voltage on DMM1 or DMM2"
- moved on the sheet: DMM1, DMM2
