File: Electrical/MainBoard/MainBoard_v5.sch (EAGLE design)
At the start: 117 parts, among them IC1 MEGA1284-P, IC2 MCP4922-E/SL, IC3 MCP4921-E/SN, IC4 TL074D, IC5 TL074D, IC6 FT232RL, Q1 BC140-10, Q2 BC160, Q3 BC140-10, Q4 BC160, Q5 BD239, Q6 BC547, Q7 BC557, Q8 16MHz, X1 FH12-45S-0.5SH, X2 22-23-2021, X3 PN61729-S

Commit message: Updated OutputControls and MainBoard in Electrical folder
Parts:
- removed C12, C13, C14, C15, C16, C17, C18, C19, C20, C21, C22: 4u7, rcl:C-EUC0805
- removed D3, D4: 5V, diode:ZENER-DIODESOD80C
- removed R27: 240k, OwnDevices:R-EU_R0805
- removed R28, R30: 100k, OwnDevices:R-EU_R0805
- removed R29: 150k, OwnDevices:R-EU_R0805
- removed R34: 10R, rcl:R-EU_R0805
- removed X1: FH12-45S-0.5SH, con-hirose:FH12-45S-0.5SH
- removed X2: 22-23-2021, con-molex:22-23-2021
- added JP1: PINHD-1X14, Connector:PINHD-1X14
- added JP2: PINHD-1X7, Connector:PINHD-1X7
Connections:
- net LCD_A0 renamed LCD_DC
- removed net !DDS_LDAC: IC1.(AIN0/INT2)PB2, IC2.!LDAC
- removed net +12V_VOLT: D4.C, IC1.(ADC3)PA3, R29.1, R30.2
- removed net -12V_VOLT: D3.C, IC1.(ADC2)PA2, IC5D.OUT, R28.1
- removed net BL_A: R34.2, X2-2.S
- removed net CAP1+: C15.1, X1-21.1
- removed net CAP1-: C14.2, C15.2, X1-23.1
- removed net CAP2+: C16.1, X1-27.1
- removed net CAP2-: C16.2, X1-25.1
- removed net CAP3+: C14.1, X1-19.1
- removed net LCD_A0_3V3: R40.1, R44.1, X1-7.1
- removed net MV1: C21.1, X1-37.1
- removed net MV2: C22.1, X1-43.1
- removed net N$27: IC5D.-IN, R27.1, R28.2
- removed net V1: C17.1, X1-29.1
- removed net V2: C18.1, X1-31.1
- removed net V3: C19.1, X1-33.1
- removed net VC: C20.1, X1-35.1
- removed net VOUT: C13.1, X1-17.1
- new net !IO_EXP_CS: IC1.(AIN0/INT2)PB2, JP2.5
- new net !TS_CS: IC1.(ADC3)PA3, JP1.11
- new net IO_EXP_INT: IC1.(OC2)PD7, JP2.6
- new net N$21: JP1.5, R40.1, R44.1
- new net TS_IRQ: IC1.(ADC2)PA2, JP1.14
- net !LCD_CS_3V3: now also JP1.3; no longer X1-3.1
- net +12V: no longer R29.2
- net +3V3: now also JP1.4, JP1.8; no longer C12.1, C13.2, X1-1.1, X1-13.1
- net +5V: now also JP1.1, JP2.1; no longer R34.1
- net -12V: no longer R27.2
- net GND: now also IC2.!LDAC, JP1.2, JP2.7; no longer C12.2, C17.2, C18.2, C19.2, C20.2, C21.2, C22.2, D3.A, D4.A, IC5D.+IN, R30.1, X1-15.1, X2-1.S
- net MISO: now also JP1.13, JP2.4
- net MOSI: now also JP1.12, JP2.3
- net MOSI_3V3: now also JP1.6; no longer X1-11.1
- net SCK: now also JP1.10, JP2.2
- net SCK_3V3: now also JP1.7; no longer X1-9.1
Other:
- note added: "Display / Touch"
- note added: "Output Controls"
- note added: "PS_Fgen_HW"
- note added: "The used display is a ILI9341 that is operating on 3,3V. This includes the MOSI, CLK, LCD_DC and !LCD_CS. The display has an integrated touch controller XPT2046. CAUTION: The display module was modified to operate the XPT2046 on 5V! The supply of the XPT2046 was cut and rewired to 5V directly."
- note added: "Touch"
- note added: "Unused"
- note removed: "(RST)"
- note removed: "Display Backlight"
- note removed: "PS_Fgen_HW v1.2"
- note removed: "Voltage Monitors"
- moved on the sheet: C1, DMM1, DMM1_NEG, DMM2, DMM2_NEG, IC5D, R39, R40, R41, R42, R43, R44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
