File: Electrical/OutputControls/OutputControls_v10.brd (EAGLE design)
At the start: 40 x 40 mm, 13 parts, among them IC1 MCP23008

Commit message: Updated OutputControls and MainBoard in Electrical folder
Parts:
- R1, R2, R3, R4: value 390 -> 330
Changed lines of the file:
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@@
 <layer number="155" name="FabDoc3" color="7" fill="1" visible="yes" active="yes"/>
 <layer number="199" name="Contour" color="7" fill="1" visible="yes" active="yes"/>
-<layer number="200" name="200bmp" color="7" fill="1" visible="no" active="yes"/>
+<layer number="200" name="200bmp" color="7" fill="10" visible="no" active="yes"/>
 <layer number="201" name="201bmp" color="7" fill="10" visible="yes" active="yes"/>
 <layer number="202" name="202bmp" color="7" fill="10" visible="yes" active="yes"/>
@@
 </class>
 </classes>
-<designrules name="default(39305442-2)">
+<designrules name="ownDesignRules2.edru">
 <param name="mdWireWire" value="0.35mm"/>
 <param name="mdWirePad" value="0.35mm"/>
@@
 <attribute name="VALUE" x="30.48" y="28.845" size="1.27" layer="27"/>
 </element>
-<element name="R1" library="OwnDevices" library_urn="urn:adsk.wipprod:fs.file:vf.a4uZ8vxKQaeHmtfASYy_rA" package="R0805" package3d_urn="urn:adsk.eagle:package:23553/2" value="390" x="35.56" y="12.7" smashed="yes" rot="R90">
+<element name="R1" library="OwnDevices" library_urn="urn:adsk.wipprod:fs.file:vf.a4uZ8vxKQaeHmtfASYy_rA" package="R0805" package3d_urn="urn:adsk.eagle:package:23553/2" value="330" x="35.56" y="12.7" smashed="yes" rot="R90">
 <attribute name="NAME" x="32.385" y="12.7" size="1.27" layer="25" font="vector" ratio="15"/>
 <attribute name="POPULARITY" value="86" x="35.56" y="12.7" size="1.778" layer="27" rot="R90" display="off"/>
@@
 <attribute name="VALUE" x="38.1" y="12.065" size="1.27" layer="27" rot="R90"/>
 </element>
-<element name="R2" library="OwnDevices" library_urn="urn:adsk.wipprod:fs.file:vf.a4uZ8vxKQaeHmtfASYy_rA" package="R0805" package3d_urn="urn:adsk.eagle:package:23553/2" value="390" x="35.56" y="17" smashed="yes" rot="R270">
+<element name="R2" library="OwnDevices" library_urn="urn:adsk.wipprod:fs.file:vf.a4uZ8vxKQaeHmtfASYy_rA" package="R0805" package3d_urn="urn:adsk.eagle:package:23553/2" value="330" x="35.56" y="17" smashed="yes" rot="R270">
 <attribute name="NAME" x="32.385" y="17" size="1.27" layer="25" font="vector" ratio="15"/>
 <attribute name="POPULARITY" value="86" x="35.56" y="17" size="1.778" layer="27" rot="R270" display="off"/>
@@
 <attribute name="VALUE" x="33.02" y="17.635" size="1.27" layer="27" rot="R270"/>
 </element>
-<element name="R3" library="OwnDevices" library_urn="urn:adsk.wipprod:fs.file:vf.a4uZ8vxKQaeHmtfASYy_rA" package="R0805" package3d_urn="urn:adsk.eagle:package:23553/2" value="390" x="34.29" y="26.67" smashed="yes" rot="R270">
+<element name="R3" library="OwnDevices" library_urn="urn:adsk.wipprod:fs.file:vf.a4uZ8vxKQaeHmtfASYy_rA" package="R0805" package3d_urn="urn:adsk.eagle:package:23553/2" value="330" x="34.29" y="26.67" smashed="yes" rot="R270">
 <attribute name="NAME" x="33.349" y="22.86" size="1.27" layer="25" font="vector" ratio="15"/>
 <attribute name="POPULARITY" value="86" x="34.29" y="26.67" size="1.778" layer="27" rot="R270" display="off"/>
@@
 <attribute name="VALUE" x="30.48" y="30.845" size="1.27" layer="27"/>
 </element>
-<element name="R4" library="OwnDevices" library_urn="urn:adsk.wipprod:fs.file:vf.a4uZ8vxKQaeHmtfASYy_rA" package="R0805" package3d_urn="urn:adsk.eagle:package:23553/2" value="390" x="38.1" y="26.67" smashed="yes" rot="R270">
+<element name="R4" library="OwnDevices" library_urn="urn:adsk.wipprod:fs.file:vf.a4uZ8vxKQaeHmtfASYy_rA" package="R0805" package3d_urn="urn:adsk.eagle:package:23553/2" value="330" x="38.1" y="26.67" smashed="yes" rot="R270">
 <attribute name="NAME" x="37.465" y="22.86" size="1.27" layer="25" font="vector" ratio="15"/>
 <attribute name="POPULARITY" value="86" x="38.1" y="26.67" size="1.778" layer="27" rot="R270" display="off"/>
