File: Electrical/FrontPanel/FrontPanel_v2.brd (EAGLE design)
At the start: 88 x 46 mm, 24 parts, among them SW1 EC12E_SW

Commit message: Updated FrontPanel and DMMRectifier in Electrical folder
Other:
- board text added: "PS_Fgen_HW FrontPanel"
- board text removed: "PS_Fgen_HW FrontPanel v1.2"
Changed lines of the file:
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@@
 <?xml version="1.0" encoding="utf-8"?>
 <!DOCTYPE eagle SYSTEM "eagle.dtd">
-<eagle version="9.6.2">
+<eagle version="9.7.0">
 <drawing>
 <settings>
-<setting alwaysvectorfont="yes"/>
+<setting alwaysvectorfont="no"/>
 <setting verticaltext="up"/>
 </settings>
@@
 <layer number="97" name="Info" color="7" fill="1" visible="no" active="no"/>
 <layer number="98" name="Guide" color="6" fill="1" visible="no" active="no"/>
-<layer number="99" name="SpiceOrder" color="5" fill="1" visible="no" active="no"/>
+<layer number="99" name="SpiceOrder" color="7" fill="1" visible="no" active="no"/>
 </layers>
 <board>
-<fusionsync huburn="a.YnVzaW5lc3M6bXlnbXgxMjQ4OA" projecturn="a.YnVzaW5lc3M6bXlnbXgxMjQ4OCNEMjAyMDAxMTAyNTQwMjAxNTE" f3durn="urn:adsk.wipprod:dm.lineage:h1ckcWdnRVyiVBv4xqEomw" pcbguid="a576bdb0-0f75-47d6-a048-163db8abff98" lastpulledtime="" lastsyncedchangeguid="f93fa148-d73c-a696-6ecf-d27c6a475278" latestrevisionid="" lastsyncedrevisionid="" lastboardhashguid="0a757cab-1d26-2fee-852c-39589efafcbf" lastpushedtime="2021-06-03T19:40:21Z" linktopcb3d="false"/>
+<fusionsync huburn="a.YnVzaW5lc3M6bXlnbXgxMjQ4OA" projecturn="a.YnVzaW5lc3M6bXlnbXgxMjQ4OCNEMjAyMDAxMTAyNTQwMjAxNTE" f3durn="urn:adsk.wipprod:dm.lineage:h1ckcWdnRVyiVBv4xqEomw" pcbguid="a576bdb0-0f75-47d6-a048-163db8abff98" lastpulledtime="" lastsyncedchangeguid="f93fa148-d73c-a696-6ecf-d27c6a475278"/>
 <plain>
 <wire x1="0" y1="0" x2="88" y2="0" width="0" layer="20"/>
@@
 <text x="55.88" y="5.715" size="1.778" layer="22" rot="MR0">NC</text>
 <text x="62.23" y="44.45" size="1.778" layer="21" align="top-left">PS_Fgen_HW
-FrontPanel
-v1.2</text>
+FrontPanel</text>
 </plain>
 <attributes>
@@
 </class>
 </classes>
-<designrules name="default">
+<designrules name="Fusion Electronics Design Rules">
+<param name="mdWireWire" value="6mil"/>
+<param name="mdWirePad" value="6mil"/>
+<param name="mdWireVia" value="6mil"/>
+<param name="mdPadPad" value="6mil"/>
+<param name="mdPadVia" value="6mil"/>
+<param name="mdViaVia" value="6mil"/>
+<param name="mdSmdPad" value="6mil"/>
+<param name="mdSmdVia" value="6mil"/>
+<param name="mdSmdSmd" value="6mil"/>
+<param name="mdCopperDimension" value="40mil"/>
+<param name="mdDrill" value="6mil"/>
+<param name="msWidth" value="6mil"/>
+<param name="msDrill" value="0.35mm"/>
+<param name="dpMaxLengthDifference" value="10mm"/>
+<param name="dpGapFactor" value="2.5"/>
 <description language="de">&lt;b&gt;EAGLE Design Rules&lt;/b&gt;
 &lt;p&gt;
@@
 <param name="mtCopper" value="0.035mm 0.035mm 0.035mm 0.035mm 0.035mm 0.035mm 0.035mm 0.035mm 0.035mm 0.035mm 0.035mm 0.035mm 0.035mm 0.035mm 0.035mm 0.035mm"/>
 <param name="mtIsolate" value="1.5mm 0.15mm 0.2mm 0.15mm 0.2mm 0.15mm 0.2mm 0.15mm 0.2mm 0.15mm 0.2mm 0.15mm 0.2mm 0.15mm 0.2mm"/>
-<param name="mdWireWire" value="6mil"/>
-<param name="mdWirePad" value="6mil"/>
-<param name="mdWireVia" value="6mil"/>
-<param name="mdPadPad" value="6mil"/>
-<param name="mdPadVia" value="6mil"/>
-<param name="mdViaVia" value="6mil"/>
-<param name="mdSmdPad" value="6mil"/>
-<param name="mdSmdVia" value="6mil"/>
-<param name="mdSmdSmd" value="6mil"/>
 <param name="mdViaViaSameLayer" value="6mil"/>
 <param name="mnLayersViaInSmd" value="2"/>
-<param name="mdCopperDimension" value="40mil"/>
-<param name="mdDrill" value="6mil"/>
 <param name="mdSmdStop" value="0mil"/>
-<param name="msWidth" value="6mil"/>
-<param name="msDrill" value="0.35mm"/>
 <param name="msMicroVia" value="9.99mm"/>
 <param name="msBlindViaRatio" value="0.5"/>
@@
 <param name="slThermalIsolate" value="10mil"/>
 <param name="slThermalsForVias" value="0"/>
-<param name="dpMaxLengthDifference" value="10mm"/>
-<param name="dpGapFactor" value="2.5"/>
 <param name="checkAngle" value="0"/>
-<param name="checkFont" value="1"/>
 <param name="checkRestrict" value="1"/>
 <param name="checkStop" value="0"/>
@@
 <wire x1="76.75" y1="11.492" x2="76.75" y2="15" width="0.4064" layer="16"/>
 <wire x1="76.75" y1="15" x2="76.712" y2="15.036" width="0.1524" layer="16"/>
-<via x="66.294" y="9.144" extent="1-16" drill="1" diameter="1.5"/>
-<via x="66.294" y="14.224" extent="1-16" drill="1" diameter="1.5"/>
+<via x="66.294" y="9.144" extent="1-16" drill="1" diameter="1.5">
+</via>
+<via x="66.294" y="14.224" extent="1-16" drill="1" diameter="1.5">
+</via>
 <wire x1="66.294" y1="14.224" x2="66.226" y2="14.292" width="0.4064" layer="16"/>
 <wire x1="66.294" y1="14.224" x2="66.294" y2="9.144" width="0.4064" layer="1"/>
-<polygon width="0.4064" layer="16" isolate="0.6096" orphans="yes">
+<polygon width="0.4064" layer="16" spacing="1.27" pour="solid" isolate="0.6096" orphans="yes" thermals="yes">
+<vertex x="0" y="0"/>
+<vertex x="88.265" y="0"/>
+<vertex x="88.265" y="46.355"/>
 <vertex x="0" y="46.355"/>
-<vertex x="88.265" y="46.355"/>
-<vertex x="88.265" y="0"/>
-<vertex x="0" y="0"/>
 </polygon>
 </signal>
@@
 <wire x1="55.88" y1="11.684" x2="57.658" y2="11.684" width="0.4064" layer="16"/>
 <wire x1="55.88" y1="11.684" x2="53.428" y2="9.358396875" width="0.4064" layer="16"/>
-<via x="82.296" y="13.462" extent="1-16" drill="1" diameter="1.5"/>
-<via x="82.296" y="9.017" extent="1-16" drill="1" diameter="1.5"/>
+<via x="82.296" y="13.462" extent="1-16" drill="1" diameter="1.5">
+</via>
+<via x="82.296" y="9.017" extent="1-16" drill="1" diameter="1.5">
+</via>
 <wire x1="82.296" y1="13.462" x2="82.296" y2="9.017" width="0.4064" layer="1"/>
 <wire x1="82.266" y1="13.492" x2="82.296" y2="13.462" width="0.4064" layer="16"/>
@@
 <mfgpreviewcolor name="substratecolor" color="0xFF786E46"/>
 </mfgpreviewcolors>
+<errors>
+</errors>
 </board>
 </drawing>
