File: Electrical/FrontPanel/FrontPanel_v2.sch (EAGLE design)
At the start: 24 parts, among them SW1 EC12E_SW

Commit message: Updated FrontPanel and DMMRectifier in Electrical folder
Other:
- note added: "PS_Fgen_HW"
- note removed: "PS_Fgen_HW v1.2"
